File: BEP-RFID-cashdrawer.kicad_sch (KiCad schematic)
At the start: 5 parts, among them J1 Conn_01x08, J2 Conn_01x03, J3 Conn_01x02, J4 Conn_01x02

Commit message: update
Parts:
- added J5: Conn_01x02, Connector_PinHeader_2.54mm:PinHeader_1x02_P2.54mm_Vertical, symbol PCM_4ms_Connector:Conn_01x02
- J1: footprint 4ms_Connector:Pins_1x08_2.54mm_TH -> Connector_PinHeader_2.54mm:PinHeader_1x08_P2.54mm_Vertical
- J2: footprint 4ms_Connector:Pins_1x03_2.54mm_TH_AudioInsRGndL -> Connector_PinHeader_2.54mm:PinHeader_1x03_P2.54mm_Vertical
- J3, J4: footprint 4ms_Connector:Pins_1x02_2.54mm_TH -> Connector_PinHeader_2.54mm:PinHeader_1x02_P2.54mm_Vertical
Connections:
- net Bypass: now also XA1.D2 (D2_INT0)
- net GND: now also J5.2 (Pin_2)
- net MISO: now also XA1.D12; no longer XA1.MISO (SPI_MISO)
- net MOSI: now also XA1.D11; no longer XA1.MOSI (SPI_MOSI)
- net RST: now also XA1.D9; no longer XA1.RST2 (SPI_RESET)
- net SCK: now also XA1.D13; no longer XA1.SCK (SPI_SCK)
- net SDA: now also XA1.D10 (D10_CS)
- net POWERIN: now reaches XA1.VIN
- net POWERIN: now also J5.1 (Pin_1)
- no-connect marks 6 -> 23
