File: BEP-RFID-cashdrawer.kicad_pcb (KiCad board)
At the start: 2 copper layers, 58.7 x 54 mm, 6 parts, among them J1 Conn_01x08, J2 Conn_01x03, J3 Conn_01x02, J4 Conn_01x02, J5 Conn_01x02

Commit message: update 2
Other:
- board text added: "JLCJLCJLCJLC"
